File: power.kicad_sch (KiCad schematic)
At the start: 3 parts, among them J3 5024940670

Commit message: fix bugs
Parts:
- added C3, C4: 10uF, Capacitor_SMD:C_0805_2012Metric, symbol Device:C_Small
- added D2: LED, LED_SMD:LED_0603_1608Metric, symbol Device:LED
- added R5: 5.1k, Resistor_SMD:R_0805_2012Metric, symbol Device:R_Small
- added U1: AMS1117-3.3, Package_TO_SOT_SMD:SOT-223-3_TabPin2, symbol Regulator_Linear:AMS1117-3.3
Connections:
- net +3.3V: now also C4.1, R5.1, U1.2 (VO)
- net +5V: now also C3.1, U1.3 (VI)
- net GND: now also C3.2, C4.2, D2.1 (K), U1.1 (GND)
- new net: D2.2 (A), R5.2
Other:
- note added: "Voltage Regulator (5V -> 3.3V)"
