File: can.kicad_sch (KiCad schematic)
At the start: 5 parts, among them J1 Conn_01x02, U2 TJA1051T

Commit message: swap CAN TX/RX
Connections:
- net RX: now also U2.4 (RXD); no longer R3.2
- net TX: now also R3.2; no longer U2.4 (RXD)
Changed lines of the file:
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@@
 		)
 	)
-	(hierarchical_label "RX"
+	(hierarchical_label "TX"
 		(shape input)
 		(at 152.4 88.9 0)
@@
 		)
 	)
-	(hierarchical_label "TX"
+	(hierarchical_label "RX"
 		(shape input)
 		(at 152.4 86.36 0)

Commit message: swap CAN TX/RX at JST connector
Connections:
- net at JP3.2 (B), U2.6 (CANL): now also J1.2 (Pin_2); no longer J1.1 (Pin_1)
- net at R2.1, U2.7 (CANH): now also J1.1 (Pin_1); no longer J1.2 (Pin_2)
Other:
- moved on the sheet: J1
Changed lines of the file:
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@@
-	(wire
-		(pts
-			(xy 73.66 95.25) (xy 73.66 88.9)
-		)
-		(stroke
-			(width 0)
-			(type default)
-		)
-	)
 	(wire
 		(pts
@@
 	(wire
 		(pts
+			(xy 87.63 88.9) (xy 87.63 95.25)
+		)
+		(stroke
+			(width 0)
+			(type default)
+		)
+	)
+	(wire
+		(pts
 			(xy 139.7 88.9) (xy 143.51 88.9)
 		)
@@
 	(wire
 		(pts
-			(xy 73.66 86.36) (xy 73.66 78.74)
-		)
-		(stroke
-			(width 0)
-			(type default)
-		)
-	)
-	(wire
-		(pts
 			(xy 93.98 95.25) (xy 93.98 93.98)
 		)
@@
 	(wire
 		(pts
-			(xy 93.98 78.74) (xy 93.98 80.01)
-		)
-		(stroke
-			(width 0)
-			(type default)
-		)
-	)
-	(wire
-		(pts
-			(xy 73.66 78.74) (xy 93.98 78.74)
+			(xy 87.63 88.9) (xy 81.28 88.9)
+		)
+		(stroke
+			(width 0)
+			(type default)
+		)
+	)
+	(wire
+		(pts
+			(xy 93.98 78.74) (xy 114.3 78.74)
+		)
+		(stroke
+			(width 0)
+			(type default)
+		)
+	)
+	(wire
+		(pts
+			(xy 81.28 86.36) (xy 87.63 86.36)
 		)
 		(stroke
@@
 	(wire
 		(pts
-			(xy 73.66 95.25) (xy 93.98 95.25)
+			(xy 87.63 95.25) (xy 93.98 95.25)
+		)
+		(stroke
+			(width 0)
+			(type default)
+		)
+	)
+	(wire
+		(pts
+			(xy 93.98 80.01) (xy 93.98 78.74)
 		)
 		(stroke
@@
 	(wire
 		(pts
-			(xy 93.98 78.74) (xy 114.3 78.74)
+			(xy 87.63 86.36) (xy 87.63 78.74)
+		)
+		(stroke
+			(width 0)
+			(type default)
+		)
+	)
+	(wire
+		(pts
+			(xy 87.63 78.74) (xy 93.98 78.74)
 		)
 		(stroke
@@
 	(symbol
 		(lib_id "Connector_Generic:Conn_01x02")
-		(at 78.74 86.36 0)
+		(at 76.2 88.9 180)
 		(unit 1)
 		(exclude_from_sim no)
@@
 		(fields_autoplaced yes)
 		(property "Reference" "J1"
-			(at 81.28 86.995 0)
-			(effects
-				(font
-					(size 1.27 1.27)
-				)
-				(justify left)
+			(at 76.2 80.01 0)
+			(effects
+				(font
+					(size 1.27 1.27)
+				)
 			)
 		)
 		(property "Value" "Conn_01x02"
-			(at 81.28 89.535 0)
-			(effects
-				(font
-					(size 1.27 1.27)
-				)
-				(justify left)
+			(at 76.2 82.55 0)
+			(effects
+				(font
+					(size 1.27 1.27)
+				)
 			)
 		)
 		(property "Footprint" "Connector_JST:JST_XH_B2B-XH-A_1x02_P2.50mm_Vertical"
-			(at 78.74 86.36 0)
+			(at 76.2 88.9 0)
 			(effects
 				(font
@@
 		)
 		(property "Datasheet" "~"
-			(at 78.74 86.36 0)
+			(at 76.2 88.9 0)
 			(effects
 				(font
@@
 		)
 		(property "Description" ""
-			(at 78.74 86.36 0)
-			(effects
-				(font
+			(at 76.2 88.9 0)
+			(effects
+				(font
